File: megadrivearcadestick.kicad_pcb (KiCad board)
At the start: 2 copper layers, 28 parts, among them J1 Left GND, J10 B, J11 C, J12 Start, J13 Up, J14 Up GND, J15 Down, J16 Down GND, J17 DB9_Female_MountingHoles, J2 Right GND, J3 A GND, J4 B GND, J5 C GND, J6 Start GND, J7 Left, J8 Right, J9 A, U1 74LS157

Commit message: Labels
Parts:
- removed J10: B, Connector_PinHeader_2.54mm:PinHeader_1x01_P2.54mm_Horizontal
- removed J11: C, Connector_PinHeader_2.54mm:PinHeader_1x01_P2.54mm_Horizontal
- removed J12: Start, Connector_PinHeader_2.54mm:PinHeader_1x01_P2.54mm_Horizontal
- removed J13: Up, Connector_PinHeader_2.54mm:PinHeader_1x01_P2.54mm_Horizontal
- removed J14: Up GND, Connector_PinHeader_2.54mm:PinHeader_1x01_P2.54mm_Horizontal
- removed J15: Down, Connector_PinHeader_2.54mm:PinHeader_1x01_P2.54mm_Horizontal
- removed J16: Down GND, Connector_PinHeader_2.54mm:PinHeader_1x01_P2.54mm_Horizontal
- removed J17: DB9_Female_MountingHoles, footprints:DB_9F
- removed J4: B GND, Connector_PinHeader_2.54mm:PinHeader_1x01_P2.54mm_Horizontal
- removed J5: C GND, Connector_PinHeader_2.54mm:PinHeader_1x01_P2.54mm_Horizontal
- removed J6: Start GND, Connector_PinHeader_2.54mm:PinHeader_1x01_P2.54mm_Horizontal
- removed J7: Left, Connector_PinHeader_2.54mm:PinHeader_1x01_P2.54mm_Horizontal
- removed J8: Right, Connector_PinHeader_2.54mm:PinHeader_1x01_P2.54mm_Horizontal
- removed J9: A, Connector_PinHeader_2.54mm:PinHeader_1x01_P2.54mm_Horizontal
- removed R2, R3, R4, R5, R6, R7, R8, R9: 10K, Resistor_THT:R_Axial_DIN0204_L3.6mm_D1.6mm_P7.62mm_Horizontal
- added REF**: MountingHole_4.3mm_M4, MountingHole:MountingHole_4.3mm_M4, F.Cu at (105.0, 65.0)
- added REF**: MountingHole_4.3mm_M4, MountingHole:MountingHole_4.3mm_M4, F.Cu at (175.0, 65.0)
- added REF**: MountingHole_4.3mm_M4, MountingHole:MountingHole_4.3mm_M4, F.Cu at (105.0, 115.0)
- added REF**: MountingHole_4.3mm_M4, MountingHole:MountingHole_4.3mm_M4, F.Cu at (175.0, 115.0)
- added RN1: 10K, Resistor_THT:R_Array_SIP5, F.Cu at (146.0, 99.0)
- added RN2: 10K, Resistor_THT:R_Array_SIP5, F.Cu at (146.2, 71.8)
- J1: value Left GND -> CTRL Grounds; footprint Connector_PinHeader_2.54mm:PinHeader_1x01_P2.54mm_Horizontal -> footprints:PinHeader_1x09_ModSilkS
- J2: value Right GND -> CTRL; footprint Connector_PinHeader_2.54mm:PinHeader_1x01_P2.54mm_Horizontal -> footprints:PinHeader_1x09_ModSilkS
- J3: value A GND -> DB9_Female_MountingHoles; footprint Connector_PinHeader_2.54mm:PinHeader_1x01_P2.54mm_Horizontal -> footprints:DB_9F
- moved J3 66.5 mm to (102.0, 90.4), turned to 270 degrees
- moved R1 59.5 mm to (131.6, 77.3), turned to 180 degrees
- moved C1 57.4 mm to (137.8, 83.3), turned to 270 degrees
- moved J2 35.2 mm to (161.3, 100.3), turned to 180 degrees
- moved U1 24.5 mm to (124.0, 83.7)
- moved J1 23.7 mm to (170.0, 100.3), turned to 180 degrees
Connections:
- C1 pad 1: Net-(C1-Pad1) -> 5V
- J2 pad 1: GND -> LEFT
- J3 pad 1: GND -> UP
- R1 pad 1: Net-(C1-Pad1) -> 5V
- R1 pad 2: Net-(J15-Pad1) -> Net-(J3-Pad7)
- U1 pad 1: Net-(J17-Pad7) -> Net-(J3-Pad7)
- U1 pad 10: Net-(J10-Pad1) -> B
- U1 pad 11: Net-(J9-Pad1) -> A
- U1 pad 12: Net-(J17-Pad9) -> CSTART_OUT
- U1 pad 13: Net-(J11-Pad1) -> C
- U1 pad 14: Net-(J12-Pad1) -> START
- U1 pad 16: Net-(C1-Pad1) -> 5V
- U1 pad 3: Net-(J7-Pad1) -> LEFT
- U1 pad 4: Net-(J17-Pad3) -> LEFT_OUT
- U1 pad 6: Net-(J8-Pad1) -> RIGHT
- U1 pad 7: Net-(J17-Pad4) -> RIGHT_OUT
- U1 pad 9: Net-(J17-Pad6) -> AB_OUT
Routing:
- net GND: track 0.00 -> 140.2 mm, vias 0 -> 2
- net 5V: track 0.00 -> 91.6 mm
- net DOWN: track 0.00 -> 89.4 mm, vias 0 -> 1
- net UP: track 0.00 -> 86.9 mm, vias 0 -> 2
- net LEFT: track 0.00 -> 78.6 mm, vias 0 -> 1
- net RIGHT: track 0.00 -> 75.7 mm
- net B: track 0.00 -> 32.3 mm
- net START: track 0.00 -> 30.8 mm
- net A: track 0.00 -> 30.3 mm
- net C: track 0.00 -> 30.3 mm
- net CSTART_OUT: track 0.00 -> 27.2 mm, vias 0 -> 2
- net AB_OUT: track 0.00 -> 26.9 mm
- net Net-(J3-Pad7): track 0.00 -> 26.2 mm
- net RIGHT_OUT: track 0.00 -> 18.3 mm
- net LEFT_OUT: track 0.00 -> 14.0 mm
Other:
- board outline added: 80 x 60 mm
- rule trace_min: 0.2 -> 0.1524

Commit message: better routes
Parts:
- moved J1 6.00 mm to (176.0, 100.3)
Routing:
- net GND: track 140.2 -> 153.3 mm, vias 2 -> 1
- net 5V: track 91.6 -> 82.6 mm
Other:
- board text added: "Down Up Up Start C B A LEFT RIGHT"

Commit message: better routes 2
Parts:
- moved REF** 4.00 mm to (105.0, 69.0)
- moved REF** 4.00 mm to (175.0, 69.0)
- moved REF** 4.00 mm to (105.0, 111.0)
- moved REF** 4.00 mm to (175.0, 111.0)
Routing:
- net LEFT: track 78.6 -> 75.0 mm, vias 1 -> 0
Other:
- board size 80 x 60 mm -> 80 x 52 mm
Changed lines of the file:
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@@
     (thickness 1.6)
     (drawings 5)
-    (tracks 131)
+    (tracks 130)
     (zones 0)
     (modules 12)
@@
   )
   (setup
-    (last_trace_width 0.5)
+    (last_trace_width 0.25)
     (user_trace_width 0.25)
     (user_trace_width 0.5)
@@
   )
   (module MountingHole:MountingHole_4.3mm_M4 (layer F.Cu)
-    (at 105 65)
+    (at 105 69)
     (descr "Mounting Hole 4.3mm, no annular, M4")
     (tags "mounting hole 4.3mm no annular m4")
     (attr virtual)
-    (fp_text reference REF** (at 0 -5.3) (layer F.SilkS)
+    (fp_text reference REF** (at 0 -5.3) (layer F.SilkS) hide
       (effects (font (size 1 1) (thickness 0.15)))
     )
@@
   )
   (module MountingHole:MountingHole_4.3mm_M4 (layer F.Cu)
-    (at 175 65)
+    (at 175 69)
     (descr "Mounting Hole 4.3mm, no annular, M4")
     (tags "mounting hole 4.3mm no annular m4")
     (attr virtual)
-    (fp_text reference REF** (at 0 -5.3) (layer F.SilkS)
+    (fp_text reference REF** (at 0 -5.3) (layer F.SilkS) hide
       (effects (font (size 1 1) (thickness 0.15)))
     )
@@
   )
   (module MountingHole:MountingHole_4.3mm_M4 (layer F.Cu)
-    (at 105 115)
+    (at 105 111)
     (descr "Mounting Hole 4.3mm, no annular, M4")
     (tags "mounting hole 4.3mm no annular m4")
     (attr virtual)
-    (fp_text reference REF** (at 0 -5.3) (layer F.SilkS)
+    (fp_text reference REF** (at 0 -5.3) (layer F.SilkS) hide
       (effects (font (size 1 1) (thickness 0.15)))
     )
@@
   )
   (module MountingHole:MountingHole_4.3mm_M4 (layer F.Cu)
-    (at 175 115)
+    (at 175 111)
     (descr "Mounting Hole 4.3mm, no annular, M4")
     (tags "mounting hole 4.3mm no annular m4")
     (attr virtual)
-    (fp_text reference REF** (at 0 -5.3) (layer F.SilkS)
+    (fp_text reference REF** (at 0 -5.3) (layer F.SilkS) hide
       (effects (font (size 1 1) (thickness 0.15)))
     )
@@
     (effects (font (size 1.5 1.5) (thickness 0.3)))
   )
-  (gr_line (start 100 60) (end 180 60) (layer Edge.Cuts) (width 0.05))
-  (gr_line (start 100 120) (end 180 120) (layer Edge.Cuts) (width 0.05))
-  (gr_line (start 180 60) (end 180 120) (layer Edge.Cuts) (width 0.05))
-  (gr_line (start 100 60) (end 100 120) (layer Edge.Cuts) (width 0.05))
+  (gr_line (start 100 64) (end 180 64) (layer Edge.Cuts) (width 0.05))
+  (gr_line (start 100 116) (end 180 116) (layer Edge.Cuts) (width 0.05))
+  (gr_line (start 180 64) (end 180 116) (layer Edge.Cuts) (width 0.05))
+  (gr_line (start 100 64) (end 100 116) (layer Edge.Cuts) (width 0.05))
   (segment (start 131.445 86.2584) (end 131.6482 86.2584) (width 0.25) (layer B.Cu) (net 1))
   (segment (start 124.0282 93.6752) (end 124.0282 93.8784) (width 0.25) (layer B.Cu) (net 1))
@@
   (segment (start 139.631201 73.195399) (end 124.0282 88.7984) (width 0.25) (layer B.Cu) (net 10))
   (segment (start 146.2024 76.8604) (end 147.327401 75.735399) (width 0.25) (layer B.Cu) (net 10))
-  (segment (start 146.2024 76.8604) (end 164.7444 76.8604) (width 0.25) (layer B.Cu) (net 10))
-  (via (at 166.751 78.867) (size 0.8) (drill 0.4) (layers F.Cu B.Cu) (net 10))
-  (segment (start 164.7444 76.8604) (end 166.751 78.867) (width 0.25) (layer B.Cu) (net 10))
-  (segment (start 166.751 94.8944) (end 161.3408 100.3046) (width 0.25) (layer F.Cu) (net 10))
-  (segment (start 166.751 78.867) (end 166.751 94.8944) (width 0.25) (layer F.Cu) (net 10))
+  (segment (start 146.2024 76.8604) (end 162.6108 76.8604) (width 0.25) (layer B.Cu) (net 10))
+  (segment (start 162.6108 76.8604) (end 163.8554 78.105) (width 0.25) (layer B.Cu) (net 10))
+  (segment (start 163.8554 97.79) (end 161.3408 100.3046) (width 0.25) (layer B.Cu) (net 10))
+  (segment (start 163.8554 78.105) (end 163.8554 97.79) (width 0.25) (layer B.Cu) (net 10))
   (segment (start 123.1138 90.424) (end 124.0282 91.3384) (width 0.25) (layer F.Cu) (net 11))
   (segment (start 110.3884 90.424) (end 123.1138 90.424) (width 0.25) (layer F.Cu) (net 11))

Commit message: better routes 3
Other:
- outline, holes or cut-outs redrawn
- board text added: "https://github.com/Ozzyboshi/Megadrivestick"
Changed lines of the file:
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@@
   (general
     (thickness 1.6)
-    (drawings 5)
+    (drawings 10)
     (tracks 130)
     (zones 0)
@@
     (46 B.CrtYd user)
     (47 F.CrtYd user)
-    (48 B.Fab user hide)
-    (49 F.Fab user hide)
+    (48 B.Fab user)
+    (49 F.Fab user)
   )
   (setup
@@
       (effects (font (size 1 1) (thickness 0.15)))
     )
-    (fp_text value MountingHole_4.3mm_M4 (at 0 5.3) (layer F.Fab)
+    (fp_text value MountingHole_4.3mm_M4 (at 0 5.3) (layer F.Fab) hide
       (effects (font (size 1 1) (thickness 0.15)))
     )
@@
       (effects (font (size 1 1) (thickness 0.15)))
     )
-    (fp_text value MountingHole_4.3mm_M4 (at 0 5.3) (layer F.Fab)
+    (fp_text value MountingHole_4.3mm_M4 (at 0 5.3) (layer F.Fab) hide
       (effects (font (size 1 1) (thickness 0.15)))
     )
@@
       (effects (font (size 1 1) (thickness 0.15)))
     )
-    (fp_text value MountingHole_4.3mm_M4 (at 0 5.3) (layer F.Fab)
+    (fp_text value MountingHole_4.3mm_M4 (at 0 5.3) (layer F.Fab) hide
       (effects (font (size 1 1) (thickness 0.15)))
     )
@@
       (effects (font (size 1 1) (thickness 0.15)))
     )
-    (fp_text value MountingHole_4.3mm_M4 (at 0 5.3) (layer F.Fab)
+    (fp_text value MountingHole_4.3mm_M4 (at 0 5.3) (layer F.Fab) hide
       (effects (font (size 1 1) (thickness 0.15)))
     )
@@
     )
   )
+  (gr_text https://github.com/Ozzyboshi/Megadrivestick (at 139.7762 110.5408) (layer Dwgs.User)
+    (effects (font (size 1 1) (thickness 0.15)))
+  )
+  (gr_line (start 180 115) (end 180 65) (layer Edge.Cuts) (width 0.05))
+  (gr_arc (start 179 115) (end 179 116) (angle -90) (layer Edge.Cuts) (width 0.05))
+  (gr_arc (start 179 65) (end 180 65) (angle -90) (layer Edge.Cuts) (width 0.05))
+  (gr_arc (start 101 65) (end 101 64) (angle -90) (layer Edge.Cuts) (width 0.05))
+  (gr_arc (start 101 115) (end 100 115) (angle -90) (layer Edge.Cuts) (width 0.05))
   (gr_text "Down\nUp\nUp\nStart\nC\nB\nA\nLEFT\nRIGHT\n" (at 168.5036 90.3986) (layer F.Cu)
     (effects (font (size 1.5 1.5) (thickness 0.3)))
   )
-  (gr_line (start 100 64) (end 180 64) (layer Edge.Cuts) (width 0.05))
-  (gr_line (start 100 116) (end 180 116) (layer Edge.Cuts) (width 0.05))
-  (gr_line (start 180 64) (end 180 116) (layer Edge.Cuts) (width 0.05))
-  (gr_line (start 100 64) (end 100 116) (layer Edge.Cuts) (width 0.05))
+  (gr_line (start 101 64) (end 179 64) (layer Edge.Cuts) (width 0.05))
+  (gr_line (start 101 116) (end 179 116) (layer Edge.Cuts) (width 0.05))
+  (gr_line (start 100 65) (end 100 115) (layer Edge.Cuts) (width 0.05))
   (segment (start 131.445 86.2584) (end 131.6482 86.2584) (width 0.25) (layer B.Cu) (net 1))
   (segment (start 124.0282 93.6752) (end 124.0282 93.8784) (width 0.25) (layer B.Cu) (net 1))

Commit message: better routes 4
Parts:
- J2: value CTRL -> CTRLS
Changed lines of the file:
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@@
       (effects (font (size 1 1) (thickness 0.15)))
     )
-    (fp_text value "CTRL Grounds" (at 0 22.65) (layer F.Fab)
+    (fp_text value "CTRL Grounds" (at 2.0884 25.3046) (layer F.Fab)
       (effects (font (size 1 1) (thickness 0.15)))
     )
@@
       (effects (font (size 1 1) (thickness 0.15)))
     )
-    (fp_text value CTRL (at 0 22.65) (layer F.Fab)
+    (fp_text value CTRLS (at 0.0508 25.3046) (layer F.Fab)
       (effects (font (size 1 1) (thickness 0.15)))
     )
